File: 1. Source/1. Motor_MotherBoardPCB/Motor_MotherBoard/Motor_MotherBoard.sch (KiCad schematic (older format))
At the start: 0 parts

Commit message: PCB_MotorMotherBoard
PCB_MotorMotherBoard
Changed lines of the file:
@@
 $EndDescr
 $Sheet
-S 895  770  1700 800
+S 1295 720  1700 800
 U 635EAE14
 F0 "MC5004P_1" 50
 F1 "MC5004P_1.sch" 50
+F2 "CAN+" I L 1295 1150 50
+F3 "CAN-" I L 1295 1300 50
 $EndSheet
 $Sheet
-S 2960 860  1425 805
+S 1275 1820 1425 805
 U 6360DF7C
 F0 "MC5004P_2" 50
 F1 "MC5004P_2.sch" 50
+F2 "CAN+" I L 1275 2115 50
+F3 "CAN-" I L 1275 2265 50
 $EndSheet
 $Sheet
-S 4845 1160 1575 705
+S 1285 2995 1575 705
 U 635FCDFD
 F0 "Connectors" 50
 F1 "Connectors.sch" 50
+F2 "CAN+" I L 1285 3285 50
+F3 "CAN-" I L 1285 3435 50
 $EndSheet
 $Sheet
-S 7045 1265 1325 600
+S 1260 4110 1325 600
 U 6360B141
 F0 "MCDC3002P_1" 50
 F1 "MCDC3002P_1.sch" 50
+F2 "CAN+" I L 1260 4350 50
+F3 "CAN-" I L 1260 4505 50
 $EndSheet
 $Sheet
-S 5795 2475 2155 675
+S 1245 5110 2155 675
 U 6362A5B1
 F0 "MCDC3002P_2" 50
 F1 "MCDC3002P_2.sch" 50
+F2 "CAN+" I L 1245 5485 50
+F3 "CAN-" I L 1245 5635 50
 $EndSheet
+Text Label 995  1150 2    50   ~ 0
+CAN+
+Wire Wire Line
+	995  1150 1295 1150
+Text Label 995  1300 2    50   ~ 0
+CAN-
+Wire Wire Line
+	995  1300 1295 1300
+Text Label 975  2115 2    50   ~ 0
+CAN+
+Wire Wire Line
+	975  2115 1275 2115
+Text Label 975  2265 2    50   ~ 0
+CAN-
+Wire Wire Line
+	975  2265 1275 2265
+Text Label 985  3285 2    50   ~ 0
+CAN+
+Wire Wire Line
+	985  3285 1285 3285
+Text Label 985  3435 2    50   ~ 0
+CAN-
+Wire Wire Line
+	985  3435 1285 3435
+Text Label 960  4350 2    50   ~ 0
+CAN+
+Wire Wire Line
+	960  4350 1260 4350
+Text Label 960  4505 2    50   ~ 0
+CAN-
+Wire Wire Line
+	960  4505 1260 4505
+Text Label 945  5485 2    50   ~ 0
+CAN+
+Wire Wire Line
+	945  5485 1245 5485
+Text Label 945  5635 2    50   ~ 0
+CAN-
+Wire Wire Line
+	945  5635 1245 5635
 $EndSCHEMATC
