File: 1. Source/1. Motor_MotherBoardPCB/Motor_MotherBoard/Connectors.sch (KiCad schematic (older format))
At the start: 2 parts, among them J1 Connector_JST_01x03, J2 Connector_JST_01x02

Commit message: PCB_MotorMotherBoard
PCB_MotorMotherBoard
Parts:
- added R1: 120, Resistor_THT:R_Axial_DIN0204_L3.6mm_D1.6mm_P2.54mm_Vertical, symbol Device:R
- added S1: EG1218, digikey-footprints:Switch_Slide_11.6x4mm_EG1218, symbol dk_Slide-Switches:EG1218
Connections:
- net CAN_H renamed CAN+
- net CAN+: now also S1.2
- net CAN_L renamed CAN-
- net CAN-: now also R1.1
- new net: R1.2, S1.1
- no-connect marks 0 -> 1
Changed lines of the file:
@@
 	-1   0    0    1
 $EndComp
-Text GLabel 1570 1215 0    50   Input ~ 0
-CAN_H
 $Comp
 L BC_Connectors:Connector_JST_01x03 J?
@@
 	1    0    0    -1
 $EndComp
-Text GLabel 1570 1315 0    50   Input ~ 0
-CAN_L
+$Comp
+L dk_Slide-Switches:EG1218 S1
+U 1 1 63833929
+P 3605 1355
+F 0 "S1" H 3605 1636 50  0000 C CNN
+F 1 "EG1218" H 3605 1545 50  0000 C CNN
+F 2 "digikey-footprints:Switch_Slide_11.6x4mm_EG1218" H 3805 1555 50  0001 L CNN
+F 3 "http://spec_sheets.e-switch.com/specs/P040040.pdf" H 3805 1655 60  0001 L CNN
+F 4 "EG1903-ND" H 3805 1755 60  0001 L CNN "Digi-Key_PN"
+F 5 "EG1218" H 3805 1855 60  0001 L CNN "MPN"
+F 6 "Switches" H 3805 1955 60  0001 L CNN "Category"
+F 7 "Slide Switches" H 3805 2055 60  0001 L CNN "Family"
+F 8 "http://spec_sheets.e-switch.com/specs/P040040.pdf" H 3805 2155 60  0001 L CNN "DK_Datasheet_Link"
+F 9 "/product-detail/en/e-switch/EG1218/EG1903-ND/101726" H 3805 2255 60  0001 L CNN "DK_Detail_Page"
+F 10 "SWITCH SLIDE SPDT 200MA 30V" H 3805 2355 60  0001 L CNN "Description"
+F 11 "E-Switch" H 3805 2455 60  0001 L CNN "Manufacturer"
+F 12 "Active" H 3805 2555 60  0001 L CNN "Status"
+	1    3605 1355
+	1    0    0    -1
+$EndComp
+NoConn ~ 3805 1455
+$Comp
+L Device:R R1
+U 1 1 6383475F
+P 3955 1255
+F 0 "R1" V 3748 1255 50  0000 C CNN
+F 1 "120" V 3839 1255 50  0000 C CNN
+F 2 "Resistor_THT:R_Axial_DIN0204_L3.6mm_D1.6mm_P2.54mm_Vertical" V 3885 1255 50  0001 C CNN
+F 3 "~" H 3955 1255 50  0001 C CNN
+	1    3955 1255
+	0    1    1    0
+$EndComp
+Text HLabel 1570 1215 0    50   Input ~ 0
+CAN+
+Text HLabel 1570 1315 0    50   Input ~ 0
+CAN-
+Text HLabel 3405 1355 0    50   Input ~ 0
+CAN+
+Text HLabel 4105 1255 2    50   Input ~ 0
+CAN-
 $EndSCHEMATC

Commit message: MotorMotherBoard설계완료
Parts:
- added J3: Connector_JST_01x02, Connectors_JST:JST_XH_S02B-XH-A_02x2.50mm_Angled, symbol BC_Connectors:Connector_JST_01x02
- R1: footprint Resistor_THT:R_Axial_DIN0204_L3.6mm_D1.6mm_P2.54mm_Vertical -> Resistor_THT:R_Axial_DIN0204_L3.6mm_D1.6mm_P7.62mm_Horizontal
Connections:
- net GND: now also J3.1 (Pin_1)
- net VSS: now also J3.2 (Pin_2)
Changed lines of the file:
@@
 F 0 "R1" V 3748 1255 50  0000 C CNN
 F 1 "120" V 3839 1255 50  0000 C CNN
-F 2 "Resistor_THT:R_Axial_DIN0204_L3.6mm_D1.6mm_P2.54mm_Vertical" V 3885 1255 50  0001 C CNN
+F 2 "Resistor_THT:R_Axial_DIN0204_L3.6mm_D1.6mm_P7.62mm_Horizontal" V 3885 1255 50  0001 C CNN
 F 3 "~" H 3955 1255 50  0001 C CNN
 	1    3955 1255
@@
 Text HLabel 4105 1255 2    50   Input ~ 0
 CAN-
+$Comp
+L BC_Connectors:Connector_JST_01x02 J?
+U 1 1 63844A70
+P 1780 1940
+AR Path="/635EAE14/63844A70" Ref="J?"  Part="1"
+AR Path="/635FCDFD/63844A70" Ref="J3"  Part="1"
+F 0 "J3" H 1860 1932 50  0000 L CNN
+F 1 "Connector_JST_01x02" H 1860 1841 50  0000 L CNN
+F 2 "Connectors_JST:JST_XH_S02B-XH-A_02x2.50mm_Angled" H 1780 1940 50  0001 C CNN
+F 3 "" H 1780 1940 50  0001 C CNN
+	1    1780 1940
+	1    0    0    -1
+$EndComp
+$Comp
+L power:GND #PWR?
+U 1 1 63844A76
+P 1580 1940
+AR Path="/635EAE14/63844A76" Ref="#PWR?"  Part="1"
+AR Path="/635FCDFD/63844A76" Ref="#PWR01"  Part="1"
+F 0 "#PWR01" H 1580 1690 50  0001 C CNN
+F 1 "GND" V 1585 1812 50  0000 R CNN
+F 2 "" H 1580 1940 50  0001 C CNN
+F 3 "" H 1580 1940 50  0001 C CNN
+	1    1580 1940
+	0    1    1    0
+$EndComp
+$Comp
+L power:VSS #PWR?
+U 1 1 63844A7C
+P 1580 2040
+AR Path="/635EAE14/63844A7C" Ref="#PWR?"  Part="1"
+AR Path="/635FCDFD/63844A7C" Ref="#PWR02"  Part="1"
+F 0 "#PWR02" H 1580 1890 50  0001 C CNN
+F 1 "VSS" V 1598 2168 50  0000 L CNN
+F 2 "" H 1580 2040 50  0001 C CNN
+F 3 "" H 1580 2040 50  0001 C CNN
+	1    1580 2040
+	0    -1   -1   0
+$EndComp
 $EndSCHEMATC
