File: 1. Source/1. Motor_MotherBoardPCB/Motor_MotherBoard/MC5004P_1.sch (KiCad schematic (older format))
At the start: 3 parts, among them U1 MC5004P, U3 CON_6pin_motor

Commit message: PCB_MotorMotherBoard
PCB_MotorMotherBoard
Parts:
- removed U3: CON_6pin_motor, Connector_IDC:IDC-Header_2x03_P2.54mm_Vertical, symbol BC_Connectors:CON_6pin_motor
- added CON1: CON_6pin_motor, Connector_IDC:IDC-Header_2x03_P2.54mm_Vertical, symbol BC_Connectors:CON_6pin_motor
- C2: renamed from R4; value Cap -> 220uF; footprint Resistor_THT:R_Axial_DIN0414_L11.9mm_D4.5mm_P5.08mm_Vertical -> Capacitor_THT:CP_Radial_D8.0mm_P3.50mm; symbol Device:R -> Device:C
Connections:
- net CH_A: now also CON1.6 (EncA)
- net CH_B: now also CON1.5 (EncB)
- net GND: now also CON1.3 (Gnd)
- net P_A: now also CON1.2 (A)
- net P_B: now also CON1.1 (B)
- net UDD: now also CON1.4 (Vin)
- net CAN_H renamed CAN+
- net CAN_L renamed CAN-
Changed lines of the file:
@@
 $Comp
 L power:GND #PWR0101
-U 1 1 60683B69
+U 1 1 63835891
 P 4250 3615
 F 0 "#PWR0101" H 4250 3365 50  0001 C CNN
@@
 $Comp
 L power:VSS #PWR0103
-U 1 1 6068DBE2
+U 1 1 63835893
 P 4250 3815
 F 0 "#PWR0103" H 4250 3665 50  0001 C CNN
@@
 $Comp
 L power:GND #PWR0104
-U 1 1 6068F021
+U 1 1 63835894
 P 4250 4515
 F 0 "#PWR0104" H 4250 4265 50  0001 C CNN
@@
 $Comp
 L power:GND #PWR0105
-U 1 1 6068FB0E
+U 1 1 63835895
 P 5200 3315
 F 0 "#PWR0105" H 5200 3065 50  0001 C CNN
@@
 $Comp
 L power:GND #PWR0106
-U 1 1 60690C1F
+U 1 1 63835896
 P 5200 4215
 F 0 "#PWR0106" H 5200 3965 50  0001 C CNN
@@
 $Comp
 L power:GND #PWR0107
-U 1 1 60691699
+U 1 1 63835897
 P 5200 5015
 F 0 "#PWR0107" H 5200 4765 50  0001 C CNN
@@
 CH_B
 $Comp
-L BC_Connectors:CON_6pin_motor U3
-U 1 1 60682551
+L BC_Connectors:CON_6pin_motor CON1
+U 1 1 6383588F
 P 7075 3675
-F 0 "U3" V 6650 3650 50  0000 C CNN
+F 0 "CON1" V 6650 3650 50  0000 C CNN
 F 1 "CON_6pin_motor" V 6741 3650 50  0000 C CNN
 F 2 "Connector_IDC:IDC-Header_2x03_P2.54mm_Vertical" H 7075 3775 50  0001 C CNN
@@
 $EndComp
 $Comp
-L power:GND #PWR0114
+L power:GND #PWR0108
 U 1 1 60683143
 P 6775 3675
-F 0 "#PWR0114" H 6775 3425 50  0001 C CNN
+F 0 "#PWR0108" H 6775 3425 50  0001 C CNN
 F 1 "GND" V 6780 3547 50  0000 R CNN
 F 2 "" H 6775 3675 50  0001 C CNN
@@
 CH_B
 $Comp
-L Device:R R4
+L Device:C C2
 U 1 1 606A2EB0
 P 7065 2955
-F 0 "R4" V 6858 2955 50  0000 C CNN
-F 1 "Cap" V 6949 2955 50  0000 C CNN
-F 2 "Resistor_THT:R_Axial_DIN0414_L11.9mm_D4.5mm_P5.08mm_Vertical" V 6995 2955 50  0001 C CNN
+F 0 "C2" V 6858 2955 50  0000 C CNN
+F 1 "220uF" V 6949 2955 50  0000 C CNN
+F 2 "Capacitor_THT:CP_Radial_D8.0mm_P3.50mm" V 6995 2955 50  0001 C CNN
 F 3 "~" H 7065 2955 50  0001 C CNN
 	1    7065 2955
@@
 $EndComp
 $Comp
-L power:VSS #PWR0112
+L power:VSS #PWR0109
 U 1 1 606A334B
 P 6915 2955
-F 0 "#PWR0112" H 6915 2805 50  0001 C CNN
+F 0 "#PWR0109" H 6915 2805 50  0001 C CNN
 F 1 "VSS" V 6933 3083 50  0000 L CNN
 F 2 "" H 6915 2955 50  0001 C CNN
@@
 $EndComp
 $Comp
-L power:GND #PWR0113
-U 1 1 606A3B9C
+L power:GND #PWR0110
+U 1 1 6383589A
 P 7215 2955
-F 0 "#PWR0113" H 7215 2705 50  0001 C CNN
+F 0 "#PWR0110" H 7215 2705 50  0001 C CNN
 F 1 "GND" V 7220 2827 50  0000 R CNN
 F 2 "" H 7215 2955 50  0001 C CNN
@@
 Wire Notes Line
 	5525 2545 3895 2545
-Text GLabel 5200 4815 2    50   Input ~ 0
-CAN_H
-Text GLabel 5200 4915 2    50   Input ~ 0
-CAN_L
 Wire Notes Line
 	5525 5310 5525 2560
@@
 Wire Notes Line
 	6410 2610 6410 2605
+Text HLabel 5200 4815 2    50   Input ~ 0
+CAN+
+Text HLabel 5200 4915 2    50   Input ~ 0
+CAN-
 $EndSCHEMATC

Commit message: MotorMotherBoard설계완료
Other:
- moved on the sheet: C2
Changed lines of the file:
@@
 L Device:C C2
 U 1 1 606A2EB0
-P 7065 2955
-F 0 "C2" V 6858 2955 50  0000 C CNN
-F 1 "220uF" V 6949 2955 50  0000 C CNN
-F 2 "Capacitor_THT:CP_Radial_D8.0mm_P3.50mm" V 6995 2955 50  0001 C CNN
-F 3 "~" H 7065 2955 50  0001 C CNN
-	1    7065 2955
-	0    1    1    0
+P 7040 2795
+F 0 "C2" V 6833 2795 50  0000 C CNN
+F 1 "220uF" V 6924 2795 50  0000 C CNN
+F 2 "Capacitor_THT:CP_Radial_D8.0mm_P3.50mm" V 6970 2795 50  0001 C CNN
+F 3 "~" H 7040 2795 50  0001 C CNN
+	1    7040 2795
+	0    -1   -1   0
 $EndComp
 $Comp
 L power:VSS #PWR0109
 U 1 1 606A334B
-P 6915 2955
-F 0 "#PWR0109" H 6915 2805 50  0001 C CNN
-F 1 "VSS" V 6933 3083 50  0000 L CNN
-F 2 "" H 6915 2955 50  0001 C CNN
-F 3 "" H 6915 2955 50  0001 C CNN
-	1    6915 2955
-	0    -1   -1   0
+P 7190 2795
+F 0 "#PWR0109" H 7190 2645 50  0001 C CNN
+F 1 "VSS" V 7208 2923 50  0000 L CNN
+F 2 "" H 7190 2795 50  0001 C CNN
+F 3 "" H 7190 2795 50  0001 C CNN
+	1    7190 2795
+	0    1    1    0
 $EndComp
 $Comp
 L power:GND #PWR0110
 U 1 1 6383589A
-P 7215 2955
-F 0 "#PWR0110" H 7215 2705 50  0001 C CNN
-F 1 "GND" V 7220 2827 50  0000 R CNN
-F 2 "" H 7215 2955 50  0001 C CNN
-F 3 "" H 7215 2955 50  0001 C CNN
-	1    7215 2955
-	0    -1   -1   0
+P 6890 2795
+F 0 "#PWR0110" H 6890 2545 50  0001 C CNN
+F 1 "GND" V 6895 2667 50  0000 R CNN
+F 2 "" H 6890 2795 50  0001 C CNN
+F 3 "" H 6890 2795 50  0001 C CNN
+	1    6890 2795
+	0    1    1    0
 $EndComp
 Wire Notes Line
