File: 1. Source/1. Motor_MotherBoardPCB/Motor_MotherBoard/Motor_MotherBoard.kicad_pcb (KiCad board)
At the start: 2 copper layers, 16 parts, among them CON1 CON_6pin_motor, CON2 CON_6pin_motor, CON3 CON_6pin_motor, CON4 CON_6pin_motor, J1 Connector_JST_01x03, J2 Connector_JST_01x02, U1 MC5004P, U3 MC5004P, U5 MCDC3002P, U6 MCDC3002P

Commit message: MotorMotherBoard설계완료
Parts:
- added J3: Connector_JST_01x02, Connectors_JST:JST_XH_S02B-XH-A_02x2.50mm_Angled, F.Cu at (44.1, 73.4)
- added REF**: MountingHole_3.2mm_M3, MountingHole:MountingHole_3.2mm_M3, F.Cu at (155.0, 25.0)
- added REF**: M_Hole_3.2mm_M3, MountingHole:MountingHole_3.2mm_M3, F.Cu at (40.0, 25.0)
- added REF**: MountingHole_3.2mm_M3, MountingHole:MountingHole_3.2mm_M3, F.Cu at (40.0, 105.0)
- added REF**: MountingHole_3.2mm_M3, MountingHole:MountingHole_3.2mm_M3, F.Cu at (155.0, 105.0)
- R1: footprint Resistor_THT:R_Axial_DIN0204_L3.6mm_D1.6mm_P2.54mm_Vertical -> Resistor_THT:R_Axial_DIN0204_L3.6mm_D1.6mm_P7.62mm_Horizontal
- moved J1 21.8 mm to (44.1, 92.1)
- moved J2 21.1 mm to (44.1, 59.6)
- moved C2 10.8 mm to (41.0, 45.6)
- moved U1 10.4 mm to (55.0, 64.7)
- moved U3 10.4 mm to (78.6, 64.7)
- moved CON1 10.4 mm to (52.2, 26.1)
- moved CON3 10.4 mm to (103.2, 26.1)
- moved U5 10.4 mm to (134.0, 62.6)
- moved U6 10.4 mm to (106.0, 62.6)
- moved C3 10.4 mm to (65.9, 45.6)
- moved CON4 10.4 mm to (131.2, 26.1)
- moved CON2 10.4 mm to (76.2, 26.1)
- moved C4 9.88 mm to (137.8, 94.6), turned to 90 degrees
- moved C1 9.86 mm to (109.9, 94.6), turned to 90 degrees
- moved S1 7.96 mm to (152.0, 84.2)
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Connections:
- C1 pad 1: VSS -> GND
- C1 pad 2: GND -> VSS
- C4 pad 1: VSS -> GND
- C4 pad 2: GND -> VSS
Routing:
- net VSS: track 0.00 -> 205.8 mm, vias 0 -> 2
- net /CAN-: track 0.00 -> 127.9 mm
- net /CAN+: track 0.00 -> 118.9 mm
- net /MCDC3002P_2/Vdd3: track 0.00 -> 53.1 mm
- net /MCDC3002P_1/Vdd3: track 0.00 -> 52.5 mm
- net /MC5004P_2/UDD: track 0.00 -> 52.4 mm
- net /MC5004P_2/CH_A: track 0.00 -> 51.8 mm
- net /MC5004P_1/CH_A: track 0.00 -> 50.2 mm
- net /MC5004P_1/UDD: track 0.00 -> 49.8 mm
- net /MC5004P_2/CH_B: track 0.00 -> 39.7 mm
- net /MC5004P_1/CH_B: track 0.00 -> 38.9 mm
- net /MCDC3002P_1/Motor_A3: track 0.00 -> 34.9 mm
- net /MCDC3002P_2/Motor_A3: track 0.00 -> 34.5 mm
- net /MCDC3002P_1/EncA3: track 0.00 -> 22.8 mm
- net /MCDC3002P_2/EncA3: track 0.00 -> 21.7 mm
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- added copper zone on B.Cu, net GND
- added copper zone on F.Cu, net GND
Other:
- board outline added: 136.3 x 95.1 mm
- board text added: "V1.0_22.11.28"
