File: 3. SchematicsLabraries/MC_5004P/MC_5004P.sch (KiCad schematic (older format))
At the start: 13 parts, among them J1 Connector_JST_01x03, J2 Connector_JST_01x02, J3 Connector_JST_01x03, J4 Connector_JST_01x03, J5 Connector_JST_01x02, U1 MC5004P, U2 MOLEX_5267_8, U3 CON_6pin_motor, U4 MOLEX_5267_8

Commit message: PCB_MotorMotherBoard
PCB_MotorMotherBoard
Parts:
- C1: renamed from R4; footprint Resistor_THT:R_Axial_DIN0414_L11.9mm_D4.5mm_P5.08mm_Vertical -> Capacitor_THT:CP_Radial_D8.0mm_P3.50mm; symbol Device:R -> pspice:CAP
Connections:
- net GND: no longer C1.1
- net VSS: no longer C1.2
Changed lines of the file:
@@
 $EndComp
 $Comp
-L Device:R R4
+L pspice:CAP C1
 U 1 1 606A2EB0
 P 2855 1110
-F 0 "R4" V 2648 1110 50  0000 C CNN
+F 0 "C1" V 2648 1110 50  0000 C CNN
 F 1 "Cap" V 2739 1110 50  0000 C CNN
-F 2 "Resistor_THT:R_Axial_DIN0414_L11.9mm_D4.5mm_P5.08mm_Vertical" V 2785 1110 50  0001 C CNN
+F 2 "Capacitor_THT:CP_Radial_D8.0mm_P3.50mm" V 2785 1110 50  0001 C CNN
 F 3 "~" H 2855 1110 50  0001 C CNN
 	1    2855 1110
