File: 1. Source/1. Motor_MotherBoardPCB/MCU_MotherBoard/ADC.sch (KiCad schematic (older format))
At the start: 23 parts, among them J11 Mol_5264_01X05, J12 Mol_5264_01X05, J13 Mol_5264_01X05, U21 LMC7660, U22 INA128PA, U23 INA128PA, U24 INA128PA

Commit message: Schematic finished
- change cap`s footprint to smd type
- artwork should be done.
Parts:
- added C1: 0.33uF, Capacitor_THT:C_Disc_D4.7mm_W2.5mm_P5.00mm, symbol Device:C
- added C2: 0.1uF, Capacitor_THT:C_Disc_D4.7mm_W2.5mm_P5.00mm, symbol Device:C
- added C3: 10uF, Capacitor_THT:C_Disc_D4.7mm_W2.5mm_P5.00mm, symbol Device:C
- added C4: 50uF, Capacitor_THT:C_Disc_D4.7mm_W2.5mm_P5.00mm, symbol Device:C
- added U3: REF5050, BC_IC_components:REF5050, symbol BC_IC_components:REF5050
- added U4: LM7805CT, digikey-footprints:TO-220-3, symbol dk_PMIC-Voltage-Regulators-Linear:LM7805CT_Obsolete
Connections:
- net Vref2 is gone; now on net Vref: C26.2, C27.2, U24.5 (Ref)
- net Vref3 is gone; now on net Vref: C23.2, C24.2, U23.5 (Ref)
- net GND: now also C1.1, C2.1, C3.1, C4.1, U3.4 (GND), U4.2 (GND)
- net Vref: now also C4.2, U3.6 (Vout)
- net +5V renamed +5VD
- net +5VD: now also C2.2, U4.3 (OUT)
- new net +9V: C1.2, C3.2, U3.2 (Vin), U4.1 (IN)
Other:
- note added: "Power"
- moved on the sheet: C17, U21

Commit message: MCUBoard작업
Parts:
- C1, C17: footprint Capacitor_THT:C_Disc_D4.7mm_W2.5mm_P5.00mm -> Capacitor_THT:CP_Radial_D8.0mm_P3.50mm
- C3: footprint Capacitor_THT:C_Disc_D4.7mm_W2.5mm_P5.00mm -> Capacitor_Tantalum_SMD:CP_EIA-7343-31_Kemet-D
- C4: value 50uF -> 10uF; footprint Capacitor_THT:C_Disc_D4.7mm_W2.5mm_P5.00mm -> Capacitor_Tantalum_SMD:CP_EIA-7343-31_Kemet-D
Changed lines of the file:
@@
 F 0 "C17" V 4590 2820 50  0000 L CNN
 F 1 "10uF" V 4340 2910 50  0000 L CNN
-F 2 "Capacitor_THT:C_Disc_D4.7mm_W2.5mm_P5.00mm" H 4478 2705 50  0001 C CNN
+F 2 "Capacitor_THT:CP_Radial_D8.0mm_P3.50mm" H 4478 2705 50  0001 C CNN
 F 3 "~" H 4440 2855 50  0001 C CNN
 	1    4440 2855
@@
 	1    0    0    -1
 $EndComp
-$Comp
-L Device:C C?
-U 1 1 63886F01
-P 4590 5795
-AR Path="/6387462E/63886F01" Ref="C?"  Part="1"
-AR Path="/6386F0B7/63886F01" Ref="C4"  Part="1"
-F 0 "C4" V 4740 5760 50  0000 L CNN
-F 1 "50uF" H 4305 5895 50  0000 L CNN
-F 2 "Capacitor_THT:C_Disc_D4.7mm_W2.5mm_P5.00mm" H 4628 5645 50  0001 C CNN
-F 3 "~" H 4590 5795 50  0001 C CNN
-	1    4590 5795
-	-1   0    0    1
-$EndComp
 Wire Wire Line
 	4315 5645 4590 5645
@@
 F 0 "C3" H 3155 5400 50  0000 L CNN
 F 1 "10uF" H 3085 5495 50  0000 L CNN
-F 2 "Capacitor_THT:C_Disc_D4.7mm_W2.5mm_P5.00mm" H 3408 5245 50  0001 C CNN
+F 2 "Capacitor_Tantalum_SMD:CP_EIA-7343-31_Kemet-D" H 3408 5245 50  0001 C CNN
 F 3 "~" H 3370 5395 50  0001 C CNN
 	1    3370 5395
@@
 F 0 "C1" V 2065 4110 50  0000 L CNN
 F 1 "0.33uF" H 1630 4245 50  0000 L CNN
-F 2 "Capacitor_THT:C_Disc_D4.7mm_W2.5mm_P5.00mm" H 1953 3995 50  0001 C CNN
+F 2 "Capacitor_THT:CP_Radial_D8.0mm_P3.50mm" H 1953 3995 50  0001 C CNN
 F 3 "~" H 1915 4145 50  0001 C CNN
 	1    1915 4145
@@
 Connection ~ 1915 3995
 Connection ~ 2715 3995
+$Comp
+L Device:C C?
+U 1 1 63886F01
+P 4590 5795
+AR Path="/6387462E/63886F01" Ref="C?"  Part="1"
+AR Path="/6386F0B7/63886F01" Ref="C4"  Part="1"
+F 0 "C4" V 4740 5760 50  0000 L CNN
+F 1 "10uF" H 4305 5895 50  0000 L CNN
+F 2 "Capacitor_Tantalum_SMD:CP_EIA-7343-31_Kemet-D" H 4628 5645 50  0001 C CNN
+F 3 "~" H 4590 5795 50  0001 C CNN
+	1    4590 5795
+	-1   0    0    1
+$EndComp
 $EndSCHEMATC
