File: 1. Source/1. Motor_MotherBoardPCB/MCU_MotherBoard/MCU_MotherBoard.kicad_pcb (KiCad board)
At the start: 2 copper layers, 143.5 x 137.2 mm, 45 parts, among them J1 Connector_JST_01x03, J11 Mol_5264_01X05, J12 Mol_5264_01X05, J13 Mol_5264_01X05, J8 Connector_JST_01x03, J9 Connector_JST_01x02, U1 LM7809, U14 BC_Nucleo446RE, U15 LoadCell_Click4, U16 LoadCell_Click4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

Commit message: MCU_MotherBoard마무리
Parts:
- added REF**: MH_3.2mm_M3, MountingHole:MountingHole_3.2mm_M3, F.Cu at (45.7, 151.1)
- added REF**: MH_3.2mm_M3, MountingHole:MountingHole_3.2mm_M3, F.Cu at (45.7, 24.1)
- added REF**: MH_3.2mm_M3, MountingHole:MountingHole_3.2mm_M3, F.Cu at (171.4, 24.1)
- added REF**: MH_3.2mm_M3, MountingHole:MountingHole_3.2mm_M3, F.Cu at (171.4, 151.1)
- moved U15 17.7 mm to (127.1, 146.9)
- moved C24 17.7 mm to (63.9, 117.3)
- moved U1 17.7 mm to (36.1, 136.4)
- moved U16 17.7 mm to (160.0, 146.9)
- moved U17 17.7 mm to (93.1, 146.9)
- moved R9 17.7 mm to (158.9, 92.2)
- moved U2 17.7 mm to (154.7, 111.9)
- moved C18 17.7 mm to (59.4, 48.3)
- moved C19 17.7 mm to (63.9, 68.8)
- moved C20 17.7 mm to (59.5, 68.8)
- moved C21 17.7 mm to (39.3, 105.4)
- moved C22 17.7 mm to (59.4, 98.0)
- moved C28 17.7 mm to (39.3, 89.4)
- moved C4 17.7 mm to (62.1, 125.0)
- moved J11 17.7 mm to (32.1, 78.5)
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Routing:
- net /ADC1_In4: track 22.9 -> 20.3 mm
- net /ADC/Vref: track 99.1 -> 101.4 mm
- net GND: vias 0 -> 213
- added copper zone on B.Cu, net GND
- added copper zone on F.Cu, net GND
Other:
- board size 143.5 x 137.2 mm -> 156.2 x 141 mm
- net class +5V: trace_width 0.6 -> 0.5
- net class +9V: clearance 0.7 -> 0.5; trace_width 0.6 -> 0.5

Commit message: !
Other:
- net class +5V removed
- net class +9V removed
- net class Default removed
